File: Hardware/NRF24l01.kicad_sch (KiCad schematic)
At the start: 24 parts, among them IC1 RFX2401C, J1 SMA Connector, U4 NRF24L01, Y1 Crystal(16MHZ)

Commit message: USB C changes
Parts:
- FL1: footprint 2450BP14D0100T -> Telemetry:2450BP14D0100T
Changed lines of the file:
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@@
     (property "Reference" "FL1" (id 0) (at 243.84 77.47 0))
     (property "Value" "2450BP14D0100T" (id 1) (at 243.84 80.01 0))
-    (property "Footprint" "2450BP14D0100T" (id 2) (at 234.95 78.74 0)
+    (property "Footprint" "Telemetry:2450BP14D0100T" (id 2) (at 234.95 78.74 0)
       (effects (font (size 1.27 1.27)) (justify left) hide)
     )

Commit message: Changed footprint for available one
Parts:
- C1, C2: Manufacturer_Part_Number (none) -> CBR04C220J5GACAUTO; Mouser Part Number (none) -> 80-CBR04C220J5GAUTO; Mouser Price/Stock (none) -> 1,01 zł
- C22: Manufacturer_Part_Number (none) -> C0402C221J4RACAUTO; Mouser Part Number (none) -> 80-C0402C221J4RAUTO; Mouser Price/Stock (none) -> 2,60 zł
- C3: Manufacturer_Part_Number (none) -> C0402C222J3TACAUTO; Mouser Part Number (none) -> 80-C0402C222J3TAUTO; Mouser Price/Stock (none) -> 2,45 zł
- C33: Manufacturer_Part_Number (none) -> CBR04C308B5GACAUTO; Mouser Part Number (none) -> 80-CBR04C308B5GAUTO; Mouser Price/Stock (none) -> 0,914 zł
- C4: Manufacturer_Part_Number (none) -> CBR04C479B5GACAUTO; Mouser Part Number (none) -> 80-CBR04C479B5GAUTO; Mouser Price/Stock (none) -> 0,914 zł
- C5: Manufacturer_Part_Number (none) -> CBR04C159B5GACAUTO; Mouser Part Number (none) -> 80-CBR04C159B5GAUTO; Mouser Price/Stock (none) -> 1,01 zł
- C6: Manufacturer_Part_Number (none) -> CBR04C109B5GACAUTO; Mouser Part Number (none) -> 80-CBR04C109B5GAUTO; Mouser Price/Stock (none) -> 1,01 zł
- C7: Manufacturer_Part_Number (none) -> MAASU105SB7333MFCA01; Mouser Part Number (none) -> 963-MAASU105SB7333MF; Mouser Price/Stock (none) -> 0,818 zł
- C9: Manufacturer_Part_Number (none) -> C0402C102J4GACAUTO; Mouser Part Number (none) -> 80-C0402C102J4GCAUTO; Mouser Price/Stock (none) -> 1,30 zł
- FL1: Arrow Part Number 2450BP14D0100T -> (none); Arrow Price/Stock https://www.arrow.com/en/products/2450bp14d0100t/johanson-d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 -> (none); Height 0.7 -> (none); Manufacturer_Name JOHANSON TECHNOLOGY -> (none); Mouser Price/Stock https://www.mouser.co.uk/ProductDetail/Johanson-Technology/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 -> 3,46 zł
- IC1: Height 0.6 -> (none); Manufacturer_Name Skyworks -> (none); Mouser Price/Stock https://www.mouser.co.uk/ProductDetail/Skyworks-Solutions-I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 -> 7,60 zł
- J1: Manufacturer_Name Molex -> (none); Mouser Price/Stock https://www.mouser.co.uk/ProductDetail/Molex/73251-2201?qs=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 -> 40,26 zł
- L1: Manufacturer_Part_Number (none) -> MLG1005S8N2HT000; Mouser Part Number (none) -> 810-MLG1005S8N2HT000; Mouser Price/Stock (none) -> 0,673 zł
- L2: Manufacturer_Part_Number (none) -> MLG1005S2N7BTD25; Mouser Part Number (none) -> 810-MLG1005S2N7BTD25; Mouser Price/Stock (none) -> 0,818 zł
- L3: Manufacturer_Part_Number (none) -> MHQ1005P3N9CT000; Mouser Part Number (none) -> 810-MHQ1005P3N9CT000; Mouser Price/Stock (none) -> 0,673 zł
- R1: Manufacturer_Part_Number (none) -> CQ02WGF1004TCE; Mouser Part Number (none) -> CQ0402-1M-1%; Mouser Price/Stock (none) -> 0.09261
- R2: Manufacturer_Part_Number (none) -> AR02BTCY2202; Mouser Part Number (none) -> AR0402-22K-0.1%; Mouser Price/Stock (none) -> 0.39514
- Y1: Manufacturer_Part_Number (none) -> 8Z-16.000MEEQ-T; Mouser Part Number (none) -> 717-8Z-16.000MEEQ-T; Mouser Price/Stock (none) -> 6,25 zł
